Commit message: Changed reference frame to base_link from world so that it is not attached to the world.

File: move_hand_pkg/urdf/move_hand.urdf.xacro (robot description, xacro)
@@ -47,10 +47,10 @@
         </xacro:unless>
     </xacro:unless>
-    <!--world to palm transform-->
-    <link name="world"/>
+    <!-- world to palm transform-->
+    <link name="base_link"/>
     <xacro:if value="$(arg right_hand)">
         <joint name="j_palm" type="fixed">
-        <origin xyz="0 0 0.2" rpy="1.57 0 0"/> <!--origin xyz="0 0 0.2" rpy="1.57 3.14 0""/-->
-        <parent link="world"/>
+        <origin xyz="0 0 0" rpy="1.57 0 0"/> <!-- origin xyz="0 0 0.2" rpy="1.57 3.14 0""/ -->
+        <parent link="base_link"/>
         <child link="palm"/>
         </joint>
@@ -58,6 +58,6 @@
     <xacro:unless value="$(arg right_hand)">
         <joint name="j_palm" type="fixed">
-        <origin xyz="0 0 0.2" rpy="1.57 3.14 0"/> <!--origin xyz="0 0 0.2" rpy="1.57 3.14 0""/-->
-        <parent link="world"/>
+        <origin xyz="0 0 0" rpy="1.57 3.14 0"/> <!-- origin xyz="0 0 0.2" rpy="1.57 3.14 0""/ -->
+        <parent link="base_link"/>
         <child link="palm"/>
         </joint>
