Commit message: Bugfixes
Co-authored-by: jbla20 <72883493+jbla20@users.noreply.github.com>
Co-authored-by: ToRexZ <victor.risager@hotmail.com>

File: move_hand/urdf/move_hand.urdf.xacro (robot description, xacro)
@@ -47,5 +47,5 @@
         </xacro:unless>
     </xacro:unless>
-    <!-- world to palm transform-->
+    <!-- base_link to palm transform-->
     <link name="base_link"/>
     <xacro:if value="$(arg right_hand)">

File: sim_world/urdf/hands/mia_hand_camera_launch.urdf.xacro (robot description, xacro)
@@ -45,13 +45,13 @@
     <!--world to palm transform-->
     <!-- world and world interface. Makes it convenient to move the whole environment according to the world origin -->
-    <link name="world" />
-    <link name="world_interface"/>
+    <!-- <link name="world" />
+    <link name="world_interface"/> -->
     <!-- world<->world_interface joint -->
-    <joint name="world_interface_to_world" type="fixed">
+    <!-- <joint name="world_interface_to_world" type="fixed">
         <parent link="world" />
         <child link="world_interface" />
-    </joint>
+    </joint> -->
     <!--joint between world_interface and mia hand-->
-    <xacro:if value="$(arg right_hand)">
+    <!-- <xacro:if value="$(arg right_hand)">
         <joint name="j_palm" type="fixed">
         <origin xyz="0 0 0.2" rpy="0 3.1416 0"/>
@@ -64,4 +64,20 @@
         <origin xyz="0 0 0.2" rpy="3.1416 0 0"/>
         <parent link="world_interface"/>
+        <child link="palm"/>
+        </joint>
+    </xacro:unless>  -->
+    <!-- base_link to palm transform-->
+    <link name="base_link"/>
+    <xacro:if value="$(arg right_hand)">
+        <joint name="j_palm" type="fixed">
+        <origin xyz="0 0 0" rpy="1.57 0 0"/> <!-- origin xyz="0 0 0.2" rpy="1.57 3.14 0""/ -->
+        <parent link="base_link"/>
+        <child link="palm"/>
+        </joint>
+    </xacro:if>
+    <xacro:unless value="$(arg right_hand)">
+        <joint name="j_palm" type="fixed">
+        <origin xyz="0 0 0" rpy="1.57 3.14 0"/> <!-- origin xyz="0 0 0.2" rpy="1.57 3.14 0""/ -->
+        <parent link="base_link"/>
         <child link="palm"/>
         </joint>

Commit message: Changed the finger controllers to Effort Controllers. Still need to pass controllers as parameters to move_hand.urdf.xacro

File: move_hand/urdf/move_hand.urdf.xacro (robot description, xacro)
@@ -1,5 +1,5 @@
 <?xml version="1.0"?>
-  <!-- URDF TO BE LOADED ON THE PARAMETER SERVER -->
-  <robot xmlns:xacro="http://wiki.ros.org/xacro" name="mia_hand">
+<!-- URDF TO BE LOADED ON THE PARAMETER SERVER -->
+<robot xmlns:xacro="http://wiki.ros.org/xacro" name="mia_hand">
     <!-- true it loads robot model with default config provided by default yaml file
     False it loads calibrated robot model configuaration yaml file.
@@ -11,8 +11,9 @@
     Choose the right hardware interface to use for joints based on the controllers ////
     ////////////////////////////////////////////////////////////////////////////////////-->
-    <xacro:arg name="hw_interface_thumb_fle" default="VelocityJointInterface"/>
-    <xacro:arg name="hw_interface_index_fle" default="VelocityJointInterface"/>
-    <xacro:arg name="hw_interface_mrl_fle" default="VelocityJointInterface"/>
-    <xacro:arg name="robotNamespace" default="/mia_hand"/> <!-- /mia_hand -->
+    <xacro:arg name="hw_interface_thumb_fle" default="EffortJointInterface"/>
+    <xacro:arg name="hw_interface_index_fle" default="EffortJointInterface"/>
+    <xacro:arg name="hw_interface_mrl_fle" default="EffortJointInterface"/>
+    <xacro:arg name="robotNamespace" default="/mia_hand"/>
+    <!-- /mia_hand -->
     <!-- Materials -->
     <xacro:include filename="$(find mia_hand_description)/materials/materials.xacro"/>
@@ -33,13 +34,13 @@
     <xacro:if value="$(arg default_mia_model)">
         <xacro:if value="$(arg right_hand)">
-        <xacro:mia_hand_robot />
+            <xacro:mia_hand_robot />
         </xacro:if>
         <xacro:unless value="$(arg right_hand)">
-        <xacro:mia_hand_robot_left />
+            <xacro:mia_hand_robot_left />
         </xacro:unless>
     </xacro:if>
     <xacro:unless value="$(arg default_mia_model)">
         <xacro:if value="$(arg right_hand)">
-        <xacro:mia_hand_robot joint_limits_parameters_file= '$(find mia_hand_description)/calibration/$(arg joint_limits_config_filename)' />
+            <xacro:mia_hand_robot joint_limits_parameters_file= '$(find mia_hand_description)/calibration/$(arg joint_limits_config_filename)' />
         </xacro:if>
         <xacro:unless value="$(arg right_hand)">
@@ -52,6 +53,6 @@
         <joint name="j_palm" type="fixed">
         <origin xyz="0 0 0" rpy="1.57 0 0"/> <!-- origin xyz="0 0 0.2" rpy="1.57 3.14 0""/ -->
-        <parent link="base_link"/>
-        <child link="palm"/>
+            <parent link="base_link"/>
+            <child link="palm"/>
         </joint>
     </xacro:if>
@@ -59,6 +60,6 @@
         <joint name="j_palm" type="fixed">
         <origin xyz="0 0 0" rpy="1.57 3.14 0"/> <!-- origin xyz="0 0 0.2" rpy="1.57 3.14 0""/ -->
-        <parent link="base_link"/>
-        <child link="palm"/>
+            <parent link="base_link"/>
+            <child link="palm"/>
         </joint>
     </xacro:unless>

Commit message: Removed origin

File: move_hand/urdf/move_hand.urdf.xacro (robot description, xacro)
@@ -52,5 +52,5 @@
     <xacro:if value="$(arg right_hand)">
         <joint name="j_palm" type="fixed">
-        <origin xyz="0 0 0" rpy="1.57 0 0"/> <!-- origin xyz="0 0 0.2" rpy="1.57 3.14 0""/ -->
+            <origin xyz="0 0 0" rpy="1.57 0 0"/>
             <parent link="base_link"/>
             <child link="palm"/>
@@ -59,5 +59,5 @@
     <xacro:unless value="$(arg right_hand)">
         <joint name="j_palm" type="fixed">
-        <origin xyz="0 0 0" rpy="1.57 3.14 0"/> <!-- origin xyz="0 0 0.2" rpy="1.57 3.14 0""/ -->
+            <origin xyz="0 0 0" rpy="1.57 3.14 0"/>
             <parent link="base_link"/>
             <child link="palm"/>
