Commit message: Fixed bug for wrist implementation causing crash due to missing inertials

File: sim_world/urdf/hands/mia_hand_camera_launch.urdf.xacro (robot description, xacro)
@@ -6,7 +6,7 @@
     <xacro:arg name="robotNamespace"                default="mia_hand_camera"/> <!-- /mia_hand_camera -->
     <xacro:arg name="joint_limits_config_filename"  default="joint_limits.yaml" />
-    <xacro:arg name="hw_interface_thumb_fle"        default="VelocityJointInterface"/>
-    <xacro:arg name="hw_interface_index_fle"        default="VelocityJointInterface"/>
-    <xacro:arg name="hw_interface_mrl_fle"          default="VelocityJointInterface"/>
+    <xacro:arg name="hw_interface_thumb_fle"        default="EffortJointInterface"/>
+    <xacro:arg name="hw_interface_index_fle"        default="EffortJointInterface"/>
+    <xacro:arg name="hw_interface_mrl_fle"          default="EffortJointInterface"/>
     <xacro:arg name="hw_interface_wrist_rotation"   default="EffortJointInterface"/>
     <xacro:arg name="hw_interface_wrist_exfle"      default="EffortJointInterface"/>
@@ -17,4 +17,11 @@
     <!-- Materials -->
     <xacro:include filename="$(find mia_hand_description)/materials/materials.xacro"/>
+    <!-- Wrist -->
+    <xacro:include filename="$(find sim_world)/urdf/macros/wrist_gazebo.urdf.xacro"/>
+    <xacro:wrist_gazebo hw_interface_wrist_rotation="$(arg hw_interface_wrist_rotation)"
+                        hw_interface_wrist_exfle="$(arg hw_interface_wrist_exfle)"
+                        hw_interface_wrist_ulra= "$(arg hw_interface_wrist_ulra)"
+                        robotNamespace= "$(arg robotNamespace)"
+                        LoadGZPlugin="false"/>
     <!-- Import Transmission and all Gazebo-customization elements, including Gazebo colors and teh Gazebo plugin-->
     <xacro:include filename="$(find mia_hand_description)/urdf/mia_hand_gazebo.urdf.xacro" />
@@ -22,11 +29,4 @@
                         hw_interface_index_fle="$(arg hw_interface_index_fle)"
                         hw_interface_mrl_fle= "$(arg hw_interface_mrl_fle)"
-                        robotNamespace= "$(arg robotNamespace)"
-                        LoadGZPlugin="true"/>
-    <!-- Wrist -->
-    <xacro:include filename="$(find sim_world)/urdf/macros/wrist_gazebo.urdf.xacro"/>
-    <xacro:wrist_gazebo hw_interface_wrist_rotation="$(arg hw_interface_wrist_rotation)"
-                        hw_interface_wrist_exfle="$(arg hw_interface_wrist_exfle)"
-                        hw_interface_wrist_ulra= "$(arg hw_interface_wrist_ulra)"
                         robotNamespace= "$(arg robotNamespace)"
                         LoadGZPlugin="true"/>
@@ -54,30 +54,27 @@
         </xacro:unless>
     </xacro:unless>
-    <!--world to palm transform-->
-    <!-- world and world interface. Makes it convenient to move the whole environment according to the world origin -->
-    <link name="world" />
-    <link name="world_interface"/>
-    <!-- world<->world_interface joint -->
-    <joint name="world_interface_to_world" type="fixed">
-        <parent link="world" />
-        <child link="world_interface" />
-    </joint>
-    <!--joint between world_interface and mia hand-->
+    <!-- base_link to palm transform-->
+    <link name="base_link"/>
     <xacro:if value="$(arg right_hand)">
-        <joint name="j_base_link" type="fixed">
-        <origin xyz="0 0 0.2" rpy="0 3.1416 0"/>
-        <parent link="world_interface"/>
-        <child link="base_link"/>
+        <joint name="j_palm" type="fixed">
+        <origin xyz="0 0 0" rpy="0 0 0"/> <!-- origin xyz="0 0 1" rpy="1.57 0 0""/ -->
+        <parent link="base_link"/>
+        <child link="wrist_link"/>
         </joint>
     </xacro:if>
     <xacro:unless value="$(arg right_hand)">
-        <joint name="j_base_link_interface" type="fixed">
-        <origin xyz="0 0 0.2" rpy="3.1416 0 0"/>
-        <parent link="world_interface"/>
-        <child link="base_link"/>
+        <joint name="j_palm" type="fixed">
+        <origin xyz="0 0 0" rpy="0 0 0"/> <!-- origin xyz="0 0 1" rpy="1.57 3.14 0""/ -->
+        <parent link="base_link"/>
+        <child link="wrist_link"/>
         </joint>
     </xacro:unless>
-    <!-- base_link to palm transform-->
-    <link name="base_link"/>
+    <link name="wrist_link">
+        <inertial>
+            <origin xyz="0 0 0" rpy="0 0 0"/>
+            <mass value="0.1"/>
+            <inertia ixx="0.01" ixy="0" ixz="0" iyy="0.01" iyz="0" izz="0.01"/>
+        </inertial>
+    </link>
     <xacro:if value="$(arg wrist_rotation)">
         <!-- Include the macro to read the wrist joint limits -->
@@ -89,51 +86,48 @@
         <joint name="j_wrist_rotation" type="revolute">
             <limit lower="${j_wrist_rotation_lower_limit}" upper="${j_wrist_rotation_upper_limit}" effort="1.75" velocity="3.140000105"/>
-            <origin xyz="0 0.2 0" rpy="0 0 0"/>
-            <parent link="base_link"/>
-            <child link="rot_to_exfle_link"/>
+            <origin xyz="0 0.0 0" rpy="0 0 0"/>
+            <parent link="wrist_link"/>
+            <child link="rot_link"/>
             <!-- <dynamics damping="0.0" friction="0.0"/> -->
             <axis xyz="1.0 0.0 0.0"/>
         </joint>
-        <link name="rot_to_exfle_link" />
+        <link name="rot_link">
+            <inertial>
+                <origin xyz="0 0 0" rpy="0 0 0"/>
+                <mass value="0.1"/>
+                <inertia ixx="0.01" ixy="0" ixz="0" iyy="0.01" iyz="0" izz="0.01"/>
+            </inertial>
+        </link>
         <!-- Extension (up) / flexion (down) = up/down  -->
         <joint name="j_wrist_exfle" type="revolute">
             <limit lower="${j_wrist_exfle_lower_limit}" upper="${j_wrist_exfle_upper_limit}" effort="1.75" velocity="3.140000105"/>
-            <origin xyz="0.2 0 0" rpy="0 0 0"/>
-            <parent link="rot_to_exfle_link"/>
-            <child link="exfle_to_ulra_link"/>
+            <origin xyz="0.0 0 0" rpy="0 0 0"/>
+            <parent link="rot_link"/>
+            <child link="exfle_link"/>
             <!-- <dynamics damping="0.0" friction="0.0"/> -->
-            <axis xyz="1.0 0.0 0.0"/>
+            <axis xyz="0.0 1.0 0.0"/>
         </joint>
-        <link name="exfle_to_ulra_link" />
+        <link name="exfle_link">
+            <inertial>
+                <origin xyz="0 0 0" rpy="0 0 0"/>
+                <mass value="0.1"/>
+                <inertia ixx="0.01" ixy="0" ixz="0" iyy="0.01" iyz="0" izz="0.01"/>
+            </inertial>
+        </link>
         <!-- Ulnar (outwards) / Radial (inwards)-->
         <joint name="j_wrist_ulra" type="revolute">
             <limit lower="${j_wrist_ulra_lower_limit}" upper="${j_wrist_ulra_upper_limit}" effort="1.75" velocity="3.140000105"/>
-            <origin xyz="0 0 0.2" rpy="0 0 0"/>
-            <parent link="exfle_to_ulra_link"/>
-            <child link="wrist_link"/>
+            <origin xyz="0 0 0.0" rpy="0 0 0"/>
+            <parent link="exfle_link"/>
+            <child link="palm"/>
             <!-- <dynamics damping="0.0" friction="0.0"/> -->
-            <axis xyz="1.0 0.0 0.0"/>
+            <axis xyz="0.0 0.0 1.0"/>
         </joint>
     </xacro:if>
     <xacro:unless value="$(arg wrist_rotation)">
-        <joint name="base_to_wrist" type="fixed">
+        <joint name="j_wrist" type="fixed">
             <origin xyz="0 0 0" rpy="0 0 0"/>
-            <parent link="base_link"/>
-            <child link="wrist_link"/>
-        </joint>
-    </xacro:unless>
-    <link name="wrist_link" />
-    <xacro:if value="$(arg right_hand)">
-        <joint name="j_palm" type="fixed">
-        <origin xyz="0 0 0" rpy="0 0 0"/> <!-- origin xyz="0 0 1" rpy="1.57 0 0""/ -->
-        <parent link="wrist_link"/>
-        <child link="palm"/>
-        </joint>
-    </xacro:if>
-    <xacro:unless value="$(arg right_hand)">
-        <joint name="j_palm" type="fixed">
-        <origin xyz="0 0 0" rpy="0 0 0"/> <!-- origin xyz="0 0 1" rpy="1.57 3.14 0""/ -->
-        <parent link="wrist_link"/>
-        <child link="palm"/>
+            <parent link="wrist_link"/>
+            <child link="palm"/>
         </joint>
     </xacro:unless>

File: sim_world/urdf/macros/joint_wrist.transmission.xacro (robot description, xacro)
@@ -2,5 +2,5 @@
 <robot xmlns:xacro="http://wiki.ros.org/xacro" name="mia_hand">
  <!-- Transmission macro -->
-  <xacro:macro name="joint_transmission_wrist_macro" params="joint_name trans_type hw_interface">
+  <xacro:macro name="joint_wrist_transmission_macro" params="joint_name trans_type hw_interface">
     <transmission name="${joint_name}_trans">
         <type>${trans_type}</type>

File: sim_world/urdf/macros/wrist_gazebo.urdf.xacro (robot description, xacro)
@@ -14,8 +14,8 @@
     Add transmission for every not fixed joint ////
    ////////////////////////////////////////////////////-->
-  <xacro:include filename="$(find sim_world)/urdf/macros/joint_transmission_wrist.xacro" />
-  <xacro:joint_transmission_wrist_macro joint_name="j_wrist_rotation"   trans_type="transmission_interface/SimpleTransmission"  hw_interface="${hw_interface_wrist_rotation}"/> <!-- Fake transmission-->
-  <xacro:joint_transmission_wrist_macro joint_name="j_wrist_exfle"  	trans_type="transmission_interface/SimpleTransmission"  hw_interface="${hw_interface_wrist_exfle}"/>
-  <xacro:joint_transmission_wrist_macro joint_name="j_wrist_ulra" 	    trans_type="transmission_interface/SimpleTransmission"  hw_interface="${hw_interface_wrist_ulra}"/>
+  <xacro:include filename="$(find sim_world)/urdf/macros/joint_wrist.transmission.xacro" />
+  <xacro:joint_wrist_transmission_macro joint_name="j_wrist_rotation"   trans_type="transmission_interface/SimpleTransmission"  hw_interface="${hw_interface_wrist_rotation}"/> <!-- Fake transmission-->
+  <xacro:joint_wrist_transmission_macro joint_name="j_wrist_exfle"  	trans_type="transmission_interface/SimpleTransmission"  hw_interface="${hw_interface_wrist_exfle}"/>
+  <xacro:joint_wrist_transmission_macro joint_name="j_wrist_ulra" 	    trans_type="transmission_interface/SimpleTransmission"  hw_interface="${hw_interface_wrist_ulra}"/>
   <!-- ros_control plugin -->
   <xacro:if value="${LoadGZPlugin}">
@@ -92,22 +92,13 @@
   </gazebo> -->
   <!-- Might need these: -->
-  <!-- <gazebo reference="j_index_fle">
+  <gazebo reference="j_wrist_rotation">
     <implicitSpringDamper>1</implicitSpringDamper>
   </gazebo>
-  <gazebo reference="j_little_fle">
+  <gazebo reference="j_wrist_exfle">
     <implicitSpringDamper>1</implicitSpringDamper>
   </gazebo>
-  <gazebo reference="j_mrl_fle">
+  <gazebo reference="j_wrist_ulra">
     <implicitSpringDamper>1</implicitSpringDamper>
   </gazebo>
-  <gazebo reference="j_ring_fle">
-    <implicitSpringDamper>1</implicitSpringDamper>
-  </gazebo>
-  <gazebo reference="j_thumb_fle">
-    <implicitSpringDamper>1</implicitSpringDamper>
-  </gazebo>
-  <gazebo reference="j_thumb_opp">
-    <implicitSpringDamper>1</implicitSpringDamper>
-  </gazebo> -->
 </xacro:macro>
 </robot>

Commit message: changed rotation axis to match the joint names.

File: sim_world/urdf/hands/mia_hand_camera_launch.urdf.xacro (robot description, xacro)
@@ -90,5 +90,5 @@
             <child link="rot_link"/>
             <!-- <dynamics damping="0.0" friction="0.0"/> -->
-            <axis xyz="1.0 0.0 0.0"/>
+            <axis xyz="0.0 1.0 0.0"/>
         </joint>
         <link name="rot_link">
@@ -106,5 +106,5 @@
             <child link="exfle_link"/>
             <!-- <dynamics damping="0.0" friction="0.0"/> -->
-            <axis xyz="0.0 1.0 0.0"/>
+            <axis xyz="1.0 0.0 0.0"/>
         </joint>
         <link name="exfle_link">

Commit message: Started implementing cartesian control, but did not integrate it correctly into the reinforcement learning framework.

File: sim_world/urdf/hands/mia_hand_camera_launch.urdf.xacro (robot description, xacro)
@@ -5,14 +5,21 @@
     <xacro:arg name="right_hand"                    default="true" />
     <xacro:arg name="robotNamespace"                default="mia_hand_camera"/> <!-- /mia_hand_camera -->
+    <xacro:arg name="camera_name"                   default="camera" />
+    <xacro:arg name="camera_topic_ns"               default="camera" />
+    <!-- Fingers -->
     <xacro:arg name="joint_limits_config_filename"  default="joint_limits.yaml" />
     <xacro:arg name="hw_interface_thumb_fle"        default="EffortJointInterface"/>
     <xacro:arg name="hw_interface_index_fle"        default="EffortJointInterface"/>
     <xacro:arg name="hw_interface_mrl_fle"          default="EffortJointInterface"/>
+    <!-- Wrist -->
+    <xacro:arg name="wrist_rotation"                default="true" />
     <xacro:arg name="hw_interface_wrist_rotation"   default="EffortJointInterface"/>
     <xacro:arg name="hw_interface_wrist_exfle"      default="EffortJointInterface"/>
     <xacro:arg name="hw_interface_wrist_ulra"       default="EffortJointInterface"/>
-    <xacro:arg name="camera_name"                   default="camera" />
-    <xacro:arg name="camera_topic_ns"               default="camera" />
-    <xacro:arg name="wrist_rotation"                default="true" />
+    <!-- Cartesian -->
+    <xacro:arg name="cartesian_control"             default="true" />
+    <xacro:arg name="hw_interface_x_cart"           default="PositionJointInterface"/>
+    <xacro:arg name="hw_interface_y_cart"           default="PositionJointInterface"/>
+    <xacro:arg name="hw_interface_z_cart"           default="PositionJointInterface"/>
     <!-- Materials -->
     <xacro:include filename="$(find mia_hand_description)/materials/materials.xacro"/>
@@ -31,4 +38,11 @@
                         robotNamespace= "$(arg robotNamespace)"
                         LoadGZPlugin="true"/>
+    <!-- Cartesian -->
+    <xacro:include filename="$(find sim_world)/urdf/macros/cartesian_gazebo.urdf.xacro"/>
+    <xacro:cartesian_gazebo hw_interface_x_cart="$(arg hw_interface_x_cart)"
+                            hw_interface_y_cart="$(arg hw_interface_y_cart)"
+                            hw_interface_z_cart="$(arg hw_interface_z_cart)"
+                            robotNamespace= "$(arg robotNamespace)"
+                            LoadGZPlugin="true"/>
     <!-- Import default robot model -->
     <xacro:if value="$(arg right_hand)">
@@ -54,4 +68,13 @@
         </xacro:unless>
     </xacro:unless>
+    <xacro:if value="$(arg cartesian_control)">
+        <!-- Fix the hand to the world -->
+        <link name="world"/>
+        <joint name="world_interface" type="fixed">
+            <origin xyz="0 0 0" rpy="0 0 0"/>
+            <parent link="world"/>
+            <child link="base_link"/>
+        </joint>
+    </xacro:if>
     <!-- base_link to palm transform-->
     <link name="base_link"/>
@@ -60,5 +83,5 @@
         <origin xyz="0 0 0" rpy="0 0 0"/> <!-- origin xyz="0 0 1" rpy="1.57 0 0""/ -->
         <parent link="base_link"/>
-        <child link="wrist_link"/>
+        <child link="cart_link"/>
         </joint>
     </xacro:if>
@@ -67,5 +90,63 @@
         <origin xyz="0 0 0" rpy="0 0 0"/> <!-- origin xyz="0 0 1" rpy="1.57 3.14 0""/ -->
         <parent link="base_link"/>
-        <child link="wrist_link"/>
+        <child link="cart_link"/>
+        </joint>
+    </xacro:unless>
+    <link name="cart_link">
+        <inertial>
+            <origin xyz="0 0 0" rpy="0 0 0"/>
+            <mass value="0.1"/>
+            <inertia ixx="0.01" ixy="0" ixz="0" iyy="0.01" iyz="0" izz="0.01"/>
+        </inertial>
+    </link>
+    <xacro:if value="$(arg cartesian_control)">
+        <!-- Include the macro to read the cartesian joint limits -->
+        <xacro:include filename="$(find sim_world)/urdf/macros/import_joint_limits_cartesian.xacro"/>
+        <!-- Read the cartesian joint limits and extract them into xacro:properties -->
+        <xacro:read_joint_limits_cartesian joint_limits_parameters_file="$(find sim_world)/urdf/calibration/joint_limits_cartesian.yaml"/>
+        <!-- x-axis -->
+        <joint name="j_x_cart" type="prismatic">
+            <limit lower="${j_x_cart_lower_limit}" upper="${j_x_cart_upper_limit}" effort="10.0" velocity="100.0"/>
+            <origin xyz="0 0.0 0" rpy="0 0 0"/>
+            <parent link="cart_link"/>
+            <child link="x_link"/>
+            <axis xyz="1.0 0.0 0.0"/>
+        </joint>
+        <link name="x_link">
+            <inertial>
+                <origin xyz="0 0 0" rpy="0 0 0"/>
+                <mass value="0.0001"/>
+                <inertia ixx="0.0001" ixy="0" ixz="0" iyy="0.0001" iyz="0" izz="0.0001"/>
+            </inertial>
+        </link>
+        <!-- y-axis -->
+        <joint name="j_y_cart" type="prismatic">
+            <limit lower="${j_y_cart_lower_limit}" upper="${j_y_cart_upper_limit}" effort="10.0" velocity="100.0"/>
+            <origin xyz="0 0.0 0" rpy="0 0 0"/>
+            <parent link="x_link"/>
+            <child link="y_link"/>
+            <axis xyz="0.0 1.0 0.0"/>
+        </joint>
+        <link name="y_link">
+            <inertial>
+                <origin xyz="0 0 0" rpy="0 0 0"/>
+                <mass value="0.0001"/>
+                <inertia ixx="0.0001" ixy="0" ixz="0" iyy="0.0001" iyz="0" izz="0.0001"/>
+            </inertial>
+        </link>
+        <!-- z-axis -->
+        <joint name="j_z_cart" type="prismatic">
+            <limit lower="${j_z_cart_lower_limit}" upper="${j_z_cart_upper_limit}" effort="10.0" velocity="100.0"/>
+            <origin xyz="0 0.0 0" rpy="0 0 0"/>
+            <parent link="y_link"/>
+            <child link="wrist_link"/>
+            <axis xyz="0.0 0.0 1.0"/>
+        </joint>
+    </xacro:if>
+    <xacro:unless value="$(arg cartesian_control)">
+        <joint name="j_cart" type="fixed">
+            <origin xyz="0 0 0" rpy="0 0 0"/>
+            <parent link="base_link"/>
+            <child link="wrist_link"/>
         </joint>
     </xacro:unless>
@@ -73,6 +154,6 @@
         <inertial>
             <origin xyz="0 0 0" rpy="0 0 0"/>
-            <mass value="0.1"/>
-            <inertia ixx="0.01" ixy="0" ixz="0" iyy="0.01" iyz="0" izz="0.01"/>
+            <mass value="0.0001"/>
+            <inertia ixx="0.0001" ixy="0" ixz="0" iyy="0.0001" iyz="0" izz="0.0001"/>
         </inertial>
     </link>
