Commit message: using velocity limits from the parameter file in the urdf.

File: sim_world/urdf/hands/mia_hand_camera_launch.urdf.xacro (robot description, xacro)
@@ -81,9 +81,9 @@
         <xacro:include filename="$(find sim_world)/urdf/macros/import_joint_limits_wrist.xacro"/>
         <!-- Read the wrist joint limits and extract them into xacro:properties -->
-        <xacro:read_joint_limits_wrist joint_limits_parameters_file="$(find sim_world)/config/joint_limits.yaml"/>
+        <xacro:read_joint_limits_wrist joint_limits_parameters_file="$(find sim_world)/config/joint_limits.yaml" hand_params_file="$(find rl_env)/params/hand/mia_hand_params.yaml"/>
         <!-- Motions for a right hand: -->
         <!-- Pronation (inwards so the palm is down) /suppination (palm up) = Rotation -->
         <joint name="j_wrist_rotation" type="revolute">
-            <limit lower="${j_wrist_rotation_lower_limit}" upper="${j_wrist_rotation_upper_limit}" effort="1.75" velocity="3.140000105"/>
+            <limit lower="${j_wrist_rotation_lower_limit}" upper="${j_wrist_rotation_upper_limit}" effort="100" velocity="${j_wrist_rotation_vel_upper_limit}"/>
             <origin xyz="0 0.0 0" rpy="0 0 0"/>
             <parent link="wrist_link"/>
@@ -101,5 +101,5 @@
         <!-- Extension (up) / flexion (down) = up/down  -->
         <joint name="j_wrist_exfle" type="revolute">
-            <limit lower="${j_wrist_exfle_lower_limit}" upper="${j_wrist_exfle_upper_limit}" effort="1.75" velocity="3.140000105"/>
+            <limit lower="${j_wrist_exfle_lower_limit}" upper="${j_wrist_exfle_upper_limit}" effort="100" velocity="${j_wrist_exfle_vel_upper_limit}"/>
             <origin xyz="0.0 0 0" rpy="0 0 0"/>
             <parent link="rot_link"/>
@@ -117,5 +117,5 @@
         <!-- Ulnar (outwards) / Radial (inwards)-->
         <joint name="j_wrist_ulra" type="revolute">
-            <limit lower="${j_wrist_ulra_lower_limit}" upper="${j_wrist_ulra_upper_limit}" effort="1.75" velocity="3.140000105"/>
+            <limit lower="${j_wrist_ulra_lower_limit}" upper="${j_wrist_ulra_upper_limit}" effort="100" velocity="${j_wrist_ulra_vel_upper_limit}"/>
             <origin xyz="0 0 0.0" rpy="0 0 0"/>
             <parent link="exfle_link"/>

File: sim_world/urdf/macros/import_joint_limits_wrist.xacro (robot description, xacro)
@@ -1,18 +1,30 @@
 <robot xmlns:xacro="http://wiki.ros.org/xacro">
-  <xacro:macro name="read_joint_limits_wrist" params="joint_limits_parameters_file">
-   <!-- Read .yaml files from disk, load content into properties -->
-   <xacro:property name="config_joint_limit_parameters" value="${xacro.load_yaml(joint_limits_parameters_file)}"/>
-   <!-- Extract subsections from yaml dictionaries -->
-   <xacro:property name="sec_limits" value="${config_joint_limit_parameters['joint_limits']}"/>
-   <!-- JOINTS LIMIT PARAMETERS -->
+  <xacro:macro name="read_joint_limits_wrist" params="joint_limits_parameters_file hand_params_file">
+    <!-- Read .yaml files from disk, load content into properties -->
+    <xacro:property name="config_joint_limit_parameters" value="${xacro.load_yaml(joint_limits_parameters_file)}"/>
+    <xacro:property name="velocity_parameter_file" value="${xacro.load_yaml(hand_params_file)}"/>
+    <!-- Extract subsections from yaml dictionaries -->
+    <xacro:property name="sec_limits" value="${config_joint_limit_parameters['joint_limits']}"/>
+    <xacro:property name="joint_velocity_limits" value="${velocity_parameter_file['general']['joint_velocity_limits']}"/>
+    <!-- JOINTS LIMIT PARAMETERS -->
     <!-- Wrist Rotation -->
-   <xacro:property name="j_wrist_rotation_lower_limit" value="${sec_limits['j_wrist_rotation']['min_position']}" scope="parent"/>
-   <xacro:property name="j_wrist_rotation_upper_limit" value="${sec_limits['j_wrist_rotation']['max_position']}" scope="parent"/>
+    <xacro:property name="j_wrist_rotation_lower_limit" value="${sec_limits['j_wrist_rotation']['min_position']}" scope="parent"/>
+    <xacro:property name="j_wrist_rotation_upper_limit" value="${sec_limits['j_wrist_rotation']['max_position']}" scope="parent"/>
     <!-- Wrist extension/flexion -->
-   <xacro:property name="j_wrist_exfle_lower_limit" value="${sec_limits['j_wrist_exfle']['min_position']}" scope="parent"/>
-   <xacro:property name="j_wrist_exfle_upper_limit" value="${sec_limits['j_wrist_exfle']['max_position']}" scope="parent"/>
-   <!-- Wrist Ulnar / Radial -->
-   <xacro:property name="j_wrist_ulra_lower_limit" value="${sec_limits['j_wrist_ulra']['min_position']}" scope="parent"/>
-   <xacro:property name="j_wrist_ulra_upper_limit" value="${sec_limits['j_wrist_ulra']['max_position']}" scope="parent"/>
+    <xacro:property name="j_wrist_exfle_lower_limit" value="${sec_limits['j_wrist_exfle']['min_position']}" scope="parent"/>
+    <xacro:property name="j_wrist_exfle_upper_limit" value="${sec_limits['j_wrist_exfle']['max_position']}" scope="parent"/>
+    <!-- Wrist Ulnar / Radial -->
+    <xacro:property name="j_wrist_ulra_lower_limit" value="${sec_limits['j_wrist_ulra']['min_position']}" scope="parent"/>
+    <xacro:property name="j_wrist_ulra_upper_limit" value="${sec_limits['j_wrist_ulra']['max_position']}" scope="parent"/>
+    <!-- JOINTS VELOCITY LIMIT PARAMETERS -->
+    <!-- Wrist Rotation -->
+    <xacro:property name="j_wrist_rotation_vel_lower_limit" value="${joint_velocity_limits['j_wrist_rotation'][0]}" scope="parent"/>
+    <xacro:property name="j_wrist_rotation_vel_upper_limit" value="${joint_velocity_limits['j_wrist_rotation'][1]}" scope="parent"/>
+    <!-- Wrist extension/flexion -->
+    <xacro:property name="j_wrist_exfle_vel_lower_limit" value="${joint_velocity_limits['j_wrist_exfle'][0]}" scope="parent"/>
+    <xacro:property name="j_wrist_exfle_vel_upper_limit" value="${joint_velocity_limits['j_wrist_exfle'][1]}" scope="parent"/>
+    <!-- Wrist Ulnar / Radial -->
+    <xacro:property name="j_wrist_ulra_vel_lower_limit" value="${joint_velocity_limits['j_wrist_ulra'][0]}" scope="parent"/>
+    <xacro:property name="j_wrist_ulra_vel_upper_limit" value="${joint_velocity_limits['j_wrist_ulra'][1]}" scope="parent"/>
  </xacro:macro>
 </robot>

Commit message: removed damping and friction

File: sim_world/urdf/hands/mia_hand_camera_launch.urdf.xacro (robot description, xacro)
@@ -89,5 +89,5 @@
             <parent link="wrist_link"/>
             <child link="rot_link"/>
-            <!-- <dynamics damping="0.0" friction="0.0"/> -->
+            <dynamics damping="0.0" friction="0.0"/>
             <axis xyz="0.0 1.0 0.0"/>
         </joint>
@@ -105,5 +105,5 @@
             <parent link="rot_link"/>
             <child link="exfle_link"/>
-            <!-- <dynamics damping="0.0" friction="0.0"/> -->
+            <dynamics damping="0.0" friction="0.0"/>
             <axis xyz="1.0 0.0 0.0"/>
         </joint>
@@ -121,5 +121,5 @@
             <parent link="exfle_link"/>
             <child link="palm"/>
-            <!-- <dynamics damping="0.0" friction="0.0"/> -->
+            <dynamics damping="0.0" friction="0.0"/>
             <axis xyz="0.0 0.0 1.0"/>
         </joint>

Commit message: Tuned the move_hand_node to make the wrist move freely.

File: sim_world/urdf/hands/mia_hand_camera_launch.urdf.xacro (robot description, xacro)
@@ -72,5 +72,5 @@
         <inertial>
             <origin xyz="0 0 0" rpy="0 0 0"/>
-            <mass value="0.1"/>
+            <mass value="0.0001"/>
             <inertia ixx="0.01" ixy="0" ixz="0" iyy="0.01" iyz="0" izz="0.01"/>
         </inertial>
@@ -94,5 +94,5 @@
             <inertial>
                 <origin xyz="0 0 0" rpy="0 0 0"/>
-                <mass value="0.1"/>
+                <mass value="0.001"/>
                 <inertia ixx="0.01" ixy="0" ixz="0" iyy="0.01" iyz="0" izz="0.01"/>
             </inertial>
@@ -110,5 +110,5 @@
             <inertial>
                 <origin xyz="0 0 0" rpy="0 0 0"/>
-                <mass value="0.1"/>
+                <mass value="0.001"/>
                 <inertia ixx="0.01" ixy="0" ixz="0" iyy="0.01" iyz="0" izz="0.01"/>
             </inertial>

Commit message: Added a lower arm visualization.

File: sim_world/urdf/hands/mia_hand_camera_launch.urdf.xacro (robot description, xacro)
@@ -16,4 +16,7 @@
     <!-- Materials -->
     <xacro:include filename="$(find mia_hand_description)/materials/materials.xacro"/>
+    <material name="B">
+      <color rgba="0.015019833 0.015019833 0.015019833 1.0"/>
+    </material>
     <!-- Wrist -->
     <xacro:include filename="$(find sim_world)/urdf/macros/wrist_gazebo.urdf.xacro"/>
@@ -76,4 +79,49 @@
         </inertial>
     </link>
+    <!-- Lower arm resemblence -->
+    <joint name="j_lower_arm" type="fixed">
+        <origin xyz="0 0 0" rpy="0 0 0"/>
+        <parent link="wrist_link"/>
+        <child link="lower_arm"/>
+    </joint>
+    <link name="lower_arm">
+        <inertial>
+            <origin xyz="0 -0.1 0" rpy="1.57079632679 0 0"/>
+            <mass value="0.01"/>
+            <inertia ixx="0.01" ixy="0" ixz="0" iyy="0.01" iyz="0" izz="0.01"/>
+        </inertial>
+        <visual>
+            <origin xyz="0 -0.1 0" rpy="1.57079632679 0 0"/>
+            <geometry>
+                <!-- <box size="0.05 0.2 0.05"/> -->
+                <cylinder radius="0.03" length="0.2"/>
+            </geometry>
+            <material name="B"/>
+            <!-- <material name="black"/> -->
+                <!-- <color rgba="0.0 0.0 0.0 1.0"/>
+            </material> -->
+        </visual>
+    </link>
+    <joint name="j_elevator" type="fixed">
+        <origin xyz="0 -0.15 0" rpy="0 0 0"/>
+        <parent link="lower_arm"/>
+        <child link="elavator"/>
+    </joint>
+    <link name="elavator">
+        <inertial>
+            <origin xyz="0 0 0" rpy="0 0 0"/>
+            <mass value="0.0001"/>
+            <inertia ixx="0.01" ixy="0" ixz="0" iyy="0.01" iyz="0" izz="0.01"/>
+        </inertial>
+        <visual>
+            <origin xyz="0 0 0" rpy="0 0 0"/>
+            <geometry>
+                <box size="0.1 0.02 0.01"/>
+            </geometry>
+            <material name="B"/>
+                <!-- <color rgba="0.0 0.0 0.0 1.0"/>
+            </material> -->
+        </visual>
+    </link>
     <xacro:if value="$(arg wrist_rotation)">
         <!-- Include the macro to read the wrist joint limits -->

Commit message: Moved camera to be under the hand
Co-authored-by: jbla20 <72883493+jbla20@users.noreply.github.com>

File: sim_world/urdf/hands/mia_hand_camera_launch.urdf.xacro (robot description, xacro)
@@ -183,10 +183,10 @@
     <xacro:if value="$(arg right_hand)">
         <xacro:sensor_d435 parent="palm" name="$(arg camera_name)" use_nominal_extrinsics="true">
-            <origin xyz="0 0 -0.05" rpy="3.1416 0 1.5708"/>
+            <origin xyz="0 0 0.04" rpy="3.1416 0 1.5708"/>
         </xacro:sensor_d435>
     </xacro:if>
     <xacro:unless value="$(arg right_hand)">
         <xacro:sensor_d435 parent="palm" name="$(arg camera_name)" use_nominal_extrinsics="true">
-            <origin xyz="0 0 -0.05" rpy="0 3.1416 1.5708"/>
+            <origin xyz="0 0 0.04" rpy="0 3.1416 1.5708"/>
         </xacro:sensor_d435>
     </xacro:unless>
